Commit message: URDF-ROS

File: src/Robot_arm_URDF/urdf/Robot_arm_URDF.urdf (robot description, URDF)
Before this commit: robot Robot_arm_URDF, 6 links, 5 joints
Links:
- added link magnet_link, mass 0.5; collision cylinder length=0.03 radius=0.025; visual cylinder length=0.03 radius=0.025
- added link world
Joints:
- added joint base_joint: type fixed, parent world, child base_link, origin xyz=0.0 0.0 0.17 rpy=0 0 0
- added joint magnet_joint: type fixed, parent link_5, child magnet_link, origin xyz=0 0 0.10 rpy=0 0 0

Commit message: Robot movimiento

File: src/Robot_arm_URDF/urdf/Robot_arm_URDF.urdf (robot description, URDF)
Before this commit: robot Robot_arm_URDF, 7 links, 6 joints
Joints:
- joint Joint_5: limit lower=0 upper=-3.142 effort=200 velocity=3 -> lower=-3.142 upper=0 effort=200 velocity=3
